Commit message: made minimal changes to urdf v2 to have tricycle kinematics and tested to work with launch v1

File: src/basic_mobile_robot/models/basic_mobile_bot_v2.urdf (robot description, URDF)
Before this commit: robot basic_mobile_bot, 6 links, 5 joints
Links:
- removed link front_caster
- added link front_steering_wheel_link; collision cylinder length=${wheel_width} radius=${wheel_radius}; visual cylinder length=${wheel_width} radius=${wheel_radius}
- added link steering_link
- added link steering_wheel_link; collision cylinder length=${wheel_width} radius=${wheel_radius}
Joints:
- removed joint caster_joint
- added joint front_steering_wheel_joint: type revolute, parent steering_wheel_link, child front_steering_wheel_link, origin xyz=0 0 0 rpy=0 0 0, axis 0 0 1, limit lower=-3.1415 upper=3.1415 effort=10 velocity=1.0
- added joint steering_joint: type fixed, parent base_link, child steering_link, origin xyz=${steering_wheel_xoff} 0 -${wheel_zoff} rpy=0 0 0
- added joint steering_wheel_joint: type revolute, parent steering_link, child steering_wheel_link, origin xyz=0 0 0 rpy=${pi/2} 0 0, axis 0 1 0, limit lower=-1.047 upper=1.047 effort=10 velocity=1.0

Commit message: made the urdf steering joint rotation direction compatible with the sdf file

File: src/basic_mobile_robot/models/basic_mobile_bot_v2.urdf (robot description, URDF)
Before this commit: robot basic_mobile_bot, 8 links, 7 joints
Joints:
- joint steering_wheel_joint: axis 0 1 0 -> 1 0 0; origin xyz=0 0 0 rpy=${pi/2} 0 0 -> xyz=0 0 0 rpy=0 ${pi/2} ${pi/2}

Commit message: made both wheels synchronized in the urdf and sdf using a rear axle link

File: src/basic_mobile_robot/models/basic_mobile_bot_v2.urdf (robot description, URDF)
Before this commit: robot basic_mobile_bot, 8 links, 7 joints
Links:
- added link rear_axle_link
Joints:
- added joint rear_axle_joint: type revolute, parent base_link, child rear_axle_link, origin xyz=${-wheel_xoff} 0 ${-wheel_zoff} rpy=0 0 0, axis 0 1 0, limit lower=-3.1415 upper=3.1415 effort=30 velocity=5.0

Commit message: created seperate links and joints in both sdf and urdf for left and right steering links to make ackermann plugin work

File: src/basic_mobile_robot/models/basic_mobile_bot_v2.urdf (robot description, URDF)
Before this commit: robot basic_mobile_bot, 9 links, 8 joints
Links:
- removed link front_steering_wheel_link
- removed link steering_link
- removed link steering_wheel_link
- added link front_left_steering_wheel_link; collision cylinder length=${wheel_width} radius=${wheel_radius}; visual cylinder length=${wheel_width} radius=${wheel_radius}
- added link front_right_steering_wheel_link; collision cylinder length=${wheel_width} radius=${wheel_radius}; visual cylinder length=${wheel_width} radius=${wheel_radius}
- added link left_steering_link
- added link left_steering_wheel_link; collision cylinder length=${wheel_width} radius=${wheel_radius}
- added link right_steering_link
- added link right_steering_wheel_link; collision cylinder length=${wheel_width} radius=${wheel_radius}
Joints:
- removed joint front_steering_wheel_joint
- removed joint steering_joint
- removed joint steering_wheel_joint
- added joint front_left_steering_wheel_joint: type revolute, parent left_steering_wheel_link, child front_left_steering_wheel_link, origin xyz=0 0 0 rpy=0 0 0, axis 0 0 1, limit lower=-3.1415 upper=3.1415 effort=10 velocity=1.0
- added joint front_right_steering_wheel_joint: type revolute, parent right_steering_wheel_link, child front_right_steering_wheel_link, origin xyz=0 0 0 rpy=0 0 0, axis 0 0 1, limit lower=-3.1415 upper=3.1415 effort=10 velocity=1.0
- added joint left_steering_joint: type fixed, parent base_link, child left_steering_link, origin xyz=${steering_wheel_xoff} 0.1 -${wheel_zoff} rpy=0 0 0
- added joint left_steering_wheel_joint: type revolute, parent left_steering_link, child left_steering_wheel_link, origin xyz=0 0 0 rpy=0 ${pi/2} ${pi/2}, axis 1 0 0, limit lower=-1.047 upper=1.047 effort=10 velocity=1.0
- added joint right_steering_joint: type fixed, parent base_link, child right_steering_link, origin xyz=${steering_wheel_xoff} -0.1 -${wheel_zoff} rpy=0 0 0
- added joint right_steering_wheel_joint: type revolute, parent right_steering_link, child right_steering_wheel_link, origin xyz=0 0 0 rpy=0 ${pi/2} ${pi/2}, axis 1 0 0, limit lower=-1.047 upper=1.047 effort=10 velocity=1.0

Commit message: Changed urdf and sdf heavily to make ackermann compatible. Got ackermann plugin to be built locally. Had to create hello world plugins to learn how to do this. toyota.sdf was created in the process of debugging the ackermann drive.

File: src/basic_mobile_robot/models/basic_mobile_bot_v2.urdf (robot description, URDF)
Before this commit: robot basic_mobile_bot, 12 links, 11 joints
Joints:
- joint left_steering_wheel_joint: axis 1 0 0 -> -1 0 0
- joint rear_axle_joint: axis 0 1 0 -> (none); limit lower=-3.1415 upper=3.1415 effort=30 velocity=5.0 -> (none); type revolute -> fixed
- joint right_steering_wheel_joint: axis 1 0 0 -> -1 0 0

Commit message: made ackermann drive plugin work with single front steering by making adding ackermann drive plugin, making the real wheel joints as revolute, and reversing the steering wheel joint axis in sdf. also made urdf consistent with sdf. no ackermann drive plugin controller and planner added yet

File: src/basic_mobile_robot/models/basic_mobile_bot_v2.urdf (robot description, URDF)
Before this commit: robot basic_mobile_bot, 9 links, 8 joints
Joints:
- joint rear_axle_joint: axis 0 1 0 -> (none); limit lower=-3.1415 upper=3.1415 effort=30 velocity=5.0 -> (none); type revolute -> fixed
- joint steering_wheel_joint: axis 1 0 0 -> -1 0 0

Commit message: edited the urdf to scale to the actual dimensions of the tow truck, base_link kept at the centre of the vehicle. This is a commit by Ailiya and was meant to be committed to the new_consolidation_ekf_off branch.

File: src/basic_mobile_robot/models/basic_mobile_bot_v2.urdf (robot description, URDF)
Before this commit: robot basic_mobile_bot, 9 links, 8 joints
Links:
- link base_link: geometry collision box size=${base_length} ${base_width} ${base_height}; visual box size=${base_length} ${base_width} ${base_height}
- link lidar_link: mass 0.114 -> 0.35; geometry collision cylinder length=0.18 radius=0.0508; visual cylinder length=0.04 radius=0.02
Joints:
- joint lidar_joint: origin xyz=0.215 0 0.13 rpy=0 0 0 -> xyz=0.65 0 1.90 rpy=0 0 0

Commit message: changed map of imc, made changes to lidar height in urdf

File: src/basic_mobile_robot/models/basic_mobile_bot_v2.urdf (robot description, URDF)
Before this commit: robot basic_mobile_bot, 9 links, 8 joints
Joints:
- joint lidar_joint: origin xyz=0.65 0 1.90 rpy=0 0 0 -> xyz=0.65 0 2.45 rpy=0 0 0

Commit message: camera in rviz and gazebo no data yet

File: src/basic_mobile_robot/models/basic_mobile_bot_v2.urdf (robot description, URDF)
Before this commit: robot basic_mobile_bot, 9 links, 8 joints
Links:
- added link camera_link, mass 0.072; collision box size=0.09 0.025 0.025; visual box size=0.09 0.025 0.025
- added link camera_link_optical
Joints:
- added joint camera_joint: type fixed, parent base_link, child camera_link, origin xyz=0.276 0 0.181 rpy=0 0.18 0
- added joint camera_optical_joint: type fixed, parent camera_link, child camera_link_optical, origin xyz=0 0 0 rpy=${-pi/2} 0 ${pi/2}

Commit message: some changes to v2 urdf

File: src/basic_mobile_robot/models/basic_mobile_bot_v2.urdf (robot description, URDF)
Before this commit: robot basic_mobile_bot, 9 links, 8 joints
Links:
- added link trailer_link; collision box size=${trailer_length} ${trailer_width} ${trailer_height}; visual box size=${trailer_length} ${trailer_width} ${trailer_height}
Joints:
- added joint trailer_joint: type continuous, parent base_link, child trailer_link, origin xyz=${-(base_length/2)} 0 0 rpy=0 0 0

Commit message: updsted sadiqas trailers

File: src/basic_mobile_robot/models/basic_mobile_bot_v2.urdf (robot description, URDF)
Before this commit: robot basic_mobile_bot, 10 links, 9 joints
Links:
- added link front_axle_link
Joints:
- added joint front_axle_joint: type fixed, parent base_link, child front_axle_link, origin xyz=${front_wheel_xoff} 0 ${-wheel_zoff} rpy=0 0 0
- joint rear_axle_joint: origin xyz=${-wheel_xoff} 0 ${-wheel_zoff} rpy=0 0 0 -> xyz=${-rear_wheel_xoff} 0 ${-wheel_zoff} rpy=0 0 0

Commit message: urdf- Sadiqah

File: src/basic_mobile_robot/models/basic_mobile_bot_v2.urdf (robot description, URDF)
Before this commit: robot basic_mobile_bot, 11 links, 10 joints
Links:
- removed link front_axle_link
- added link trailer2_link; collision box size=${-trailer_length/2} ${trailer_width} ${trailer_height}; visual box size=${trailer_length} ${trailer_width} ${trailer_height}
- link trailer_link: geometry collision box size=${-trailer_length/2} ${trailer_width} ${trailer_height}; visual box size=${trailer_length} ${trailer_width} ${trailer_height}
Joints:
- removed joint front_axle_joint
- added joint trailer2_joint: type continuous, parent trailer_link, child trailer2_link, origin xyz=${-trailer_length} 0 0 rpy=0 0 0, axis 0 0 1
- joint rear_axle_joint: origin xyz=${-rear_wheel_xoff} 0 ${-wheel_zoff} rpy=0 0 0 -> xyz=${-wheel_xoff} 0 ${-wheel_zoff} rpy=0 0 0
- joint trailer_joint: axis (none) -> 0 0 1

Commit message: new updates in package

File: src/basic_mobile_robot/models/basic_mobile_bot_v2.urdf (robot description, URDF)
Before this commit: robot basic_mobile_bot, 11 links, 10 joints
Links:
- added link depth_camera_link, mass 0.072; collision box size=0.09 0.025 0.025; visual box size=0.09 0.025 0.025
- link camera_link_optical: mass None -> 0.001
Joints:
- added joint depth_camera_joint: type fixed, parent base_link, child depth_camera_link, origin xyz=0.215 0.10 0.13 rpy=0 0 0
- joint camera_joint: origin xyz=0.276 0 0.181 rpy=0 0.18 0 -> xyz=0.215 0 0.1 rpy=0 0 0
- joint camera_optical_joint: origin xyz=0 0 0 rpy=${-pi/2} 0 ${pi/2} -> xyz=0 0 0 rpy=-1.5708 0 1.5708

Commit message: Finally depth is working and we are getting the data - Hijab

File: src/basic_mobile_robot/models/basic_mobile_bot_v2.urdf (robot description, URDF)
Before this commit: robot basic_mobile_bot, 11 links, 10 joints
Links:
- link camera_link: mass 0.072 -> None; geometry visual box size=0.010 0.03 0.03
Joints:
- joint camera_joint: origin xyz=0.276 0 0.181 rpy=0 0.18 0 -> xyz=0.305 0 0.08 rpy=0 0 0
- joint camera_optical_joint: origin xyz=0 0 0 rpy=${-pi/2} 0 ${pi/2} -> xyz=0 0 0 rpy=${-pi/2} 0 ${-pi/2}

Commit message: performed some tests, gave better results when urdf updated, we change z value of imu in urdf

File: src/basic_mobile_robot/models/basic_mobile_bot_v2.urdf (robot description, URDF)
Before this commit: robot basic_mobile_bot, 9 links, 8 joints
Joints:
- joint imu_joint: origin xyz=-0.10 0 0.05 rpy=0 0 0 -> xyz=0 0 0.71 rpy=0 0 0

Commit message: with depth points it is working using realsense camera

File: src/basic_mobile_robot/models/basic_mobile_bot_v2.urdf (robot description, URDF)
Before this commit: robot basic_mobile_bot, 9 links, 8 joints
Links:
- added link camera_link; visual box size=0.010 0.03 0.03
- added link camera_link_optical
Joints:
- added joint camera_joint: type fixed, parent base_link, child camera_link, origin xyz=0.305 0 0.08 rpy=0 0 0
- added joint camera_optical_joint: type fixed, parent camera_link, child camera_link_optical, origin xyz=0 0 0 rpy=${-pi/2} 0 ${-pi/2}

Commit message: Thurdays changes Lyeba and Hijab

File: src/basic_mobile_robot/models/basic_mobile_bot_v2.urdf (robot description, URDF)
Before this commit: robot basic_mobile_bot, 9 links, 8 joints
Joints:
- joint gps_joint: origin xyz=0.10 0 0.05 rpy=0 0 0 -> xyz=0 0 1.5 rpy=0 0 0

Commit message: pushing all the small changes

File: src/basic_mobile_robot/models/basic_mobile_bot_v2.urdf (robot description, URDF)
Before this commit: robot basic_mobile_bot, 9 links, 8 joints
Links:
- link base_link: geometry collision box size=${base_length} ${base_width+0.52} ${base_height}; visual box size=${base_length} ${base_width} ${base_height}

Commit message: increased the height of LiDAR in URDF

File: src/basic_mobile_robot/models/basic_mobile_bot_v2.urdf (robot description, URDF)
Before this commit: robot basic_mobile_bot, 9 links, 8 joints
Joints:
- joint lidar_joint: origin xyz=0.65 0 1.90 rpy=0 0 0 -> xyz=0.65 0 2.50 rpy=0 0 0

Commit message: two 2d lidars added - costmap update is buggy

File: src/basic_mobile_robot/models/basic_mobile_bot_v2.urdf (robot description, URDF)
Before this commit: robot basic_mobile_bot, 9 links, 8 joints
Links:
- added link lidar_link_2, mass 0.114; collision cylinder length=0.18 radius=0.0508; visual cylinder length=0.18 radius=0.0508
Joints:
- added joint lidar_joint_2: type fixed, parent base_link, child lidar_link_2, origin xyz=0.215 0 0.13 rpy=0 0 0

Commit message: 3D LiDAR simulation using LaserScan

File: src/basic_mobile_robot/models/basic_mobile_bot_v2.urdf (robot description, URDF)
Before this commit: robot basic_mobile_bot, 10 links, 9 joints
Links:
- removed link lidar_link_2
Joints:
- removed joint lidar_joint_2

Commit message: 2d and 3d lidar generating singlr costmap

File: src/basic_mobile_robot/models/basic_mobile_bot_v2.urdf (robot description, URDF)
Before this commit: robot basic_mobile_bot, 9 links, 8 joints
Links:
- added link lidar_link_2, mass 0.114; collision cylinder length=0.18 radius=0.0508; visual cylinder length=0.18 radius=0.0508
Joints:
- added joint lidar_joint_2: type fixed, parent base_link, child lidar_link_2, origin xyz=0.215 0 0.13 rpy=0 0 3.14159

Commit message: Fixed Rviz file

File: src/basic_mobile_robot/models/basic_mobile_bot_v2.urdf (robot description, URDF)
Before this commit: robot basic_mobile_bot, 10 links, 9 joints
Links:
- link base_link: geometry collision box size=${base_length} ${base_width} ${base_height}; visual box size=${base_length} ${base_width} ${base_height}
Joints:
- joint lidar_joint: origin xyz=0.215 0 0.13 rpy=0 0 0 -> xyz=0.815 0.38 1.7 rpy=0 0 0
- joint lidar_joint_2: origin xyz=0.215 0 0.13 rpy=0 0 3.14159 -> xyz=0.65 0 2.5 rpy=0 0 3.14159

Commit message: Gazebo simulationfixed as per Rviz

File: src/basic_mobile_robot/models/basic_mobile_bot_v2.urdf (robot description, URDF)
Before this commit: robot basic_mobile_bot, 10 links, 9 joints
Joints:
- joint lidar_joint_2: origin xyz=0.65 0 2.5 rpy=0 0 3.14159 -> xyz=0.65 0 1.90 rpy=0 0 3.14159
